File: kicad/power.kicad_sch (KiCad schematic)
At the start: 17 parts, among them J4 USB-C-16P, U5 BQ24075, U6 TLV75533PDBVR, U7 LP2985-33DBVR

Commit message: Add kicad/power.kicad_sch
Parts:
- removed BAT1: LiPo_PH2.0, Connector_JST:JST_PH_B2B-PH-K_1x02_P2.00mm_Vertical, symbol Connector:Conn_01x02_Pin
- removed C29, C30: 100nF, Capacitor_SMD:C_0402_1005Metric, symbol Device:C
- removed D1: SS14, Diode_SMD:D_SMA, symbol Device:D_Schottky
- removed D2: PRTR5V0U2X, Package_TO_SOT_SMD:SOT-363_SC-70-6, symbol Device:D_TVS
- removed F1: 500mA/6V, Fuse:Fuse_0805_2012Metric, symbol Device:Polyfuse
- removed J4: USB-C-16P, Connector_USB:USB_C_Receptacle_HRO_TYPE-C-31-M-12, symbol Connector:USB_C_Receptacle_USB2.0
- added C_1V8_IN, C_1V8_OUT: 1uF, Capacitor_SMD:C_0402_1005Metric, symbol Device:C
- added C_3V3_HF, C_ANAL_HF, C_VBUS: 100nF, Capacitor_SMD:C_0402_1005Metric, symbol Device:C
- added J1: LIPO_BAT, Connector_JST:JST_PH_S2B-PH-K_1x02_P2.00mm_Horizontal, symbol Connector:Conn_01x02_Pin
- added J2: USB_C_GCT_USB4085, Connector_USB:GCT_USB4085_MidMount_Horizontal, symbol Connector_USB:USB_C_Receptacle_GCT_USB4085
- added LED_CHG: RED_0603, LED_SMD:LED_0603_1608Metric, symbol Device:LED
- added R11, R12: 5.1k, Resistor_SMD:R_0402_1005Metric, symbol Device:R
- added R_CHG: 1k, Resistor_SMD:R_0402_1005Metric, symbol Device:R
- added U8: MIC5504-1.8YM5-TR, Package_TO_SOT_SMD:SOT-23-5, symbol Regulator_Linear:MIC5504-1.8
- C25, C26, C27, C28, C_U5_IN, C_VBAT: value 10uF/10V -> 4.7uF/10V X5R; footprint Capacitor_SMD:C_0805_2012Metric -> Capacitor_SMD:C_0603_1608Metric
- U5: value BQ24075 -> BQ24075RGTR; footprint Package_TO_SOT_SMD:SOT-23-8 -> Package_DFN_QFN:QFN-16-1EP_3x3mm_P0.5mm_EP1.65x1.65mm
- U6: value TLV75533PDBVR -> RT9193-33GB; symbol Regulator_Linear:TLV755P -> Regulator_Linear:RT9193-33
Other:
- note added: "POWER MANAGEMENT NOTES (v1.1): 1) Power tree: J2 (USB-C) → VBUS_USB (5V) → BQ24075 (charger) → VBAT (3.7V LiPo) VBAT → U6 RT9193-33GB → 3V3_MAIN (digital logic) VBAT → U7 LP2985-33 → 3V3_ANALOG (SI4732 VA/VDDO, ES7243E AVDD) 3V3_ANALOG → U8 MIC5504-1.8 → 1V8_SI4732 (SI4732 VDD) VBAT → FB1(audio_output.kicad_sch) → PVDD_FILT (MAX98357A PVDD) 2) LDO selection: [FIXED] U6: RT9193-33GB (was TLV75533P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"
- note removed: "POWER DESIGN NOTES: 1) USB 5V → F1(500mA polyfuse) → BQ24075 VCC ESD on D+/D- via D2 (PRTR5V0U2X) 2) BQ24075: - ISET: R10=2kΩ → ~445mA charge current - SYS output feeds both LDOs - VBAT to single-cell Li-Ion via D1(SS14) reverse protection - STATUS pin → GPIO for charge indicator (optional) 3) U6 TLV75533 (500mA) → 3V3_MAIN Powers: ESP32-WROVER-E, TFT, encoder logic, LEDs, USB-UART Bypass: 10uF +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"
