File: kicad/esp32_core.kicad_sch (KiCad schematic)
At the start: 21 parts, among them J5 DEBUG_UART, Q1 MMBT3904, Q2 MMBT3904, SW1 RESET, SW2 BOOT, U1 ESP32-WROVER-E, U9 CP2102N

Commit message: Add kicad/esp32_core.kicad_sch
Parts:
- C4, C5: value 10uF/6.3V -> 4.7uF/6.3V X5R; footprint Capacitor_SMD:C_0805_2012Metric -> Capacitor_SMD:C_0603_1608Metric
- C_CP2: value 10uF/10V -> 4.7uF/10V X5R; footprint Capacitor_SMD:C_0805_2012Metric -> Capacitor_SMD:C_0603_1608Metric
Other:
- note added: "ESP32-WROVER-E GPIO ASSIGNMENT (v1.1) ────────────────────────────────────────────────────── IO0 → BOOT button at power-on (pull-up R2 10k) [DUAL] → I2S_MCLK output after boot (12.288MHz MCLK) IO2 → ENCODER_A (pull-up 10k, 10nF debounce) IO4 → ENCODER_B (pull-up 10k, 10nF debounce) IO5 → ENCODER_SW (pull-up 10k) IO12 → LCD_DC strapping: keep LOW at boot IO13 → LCD_BL (PWM LEDC ch0) IO14 → LCD_RST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"
- note removed: "ESP32-WROVER-E GPIO ASSIGNMENT ────────────────────────────────────────────────────── IO0 → BOOT button (pull-up R2 10k) strapping IO2 → ENCODER_A (pull-up 10k, 10nF debounce) IO4 → ENCODER_B (pull-up 10k, 10nF debounce) IO5 → ENCODER_SW (pull-up 10k) IO12 → LCD_DC strapping: keep low at boot IO13 → LCD_BL (PWM LEDC ch0) IO14 → LCD_RST IO15 → SPI_CLK (VSPI SCLK) IO18 → I2S_BCLK IO19 → I2S_LRCK (W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"
