File: kicad/audio_output.kicad_sch (KiCad schematic)
At the start: 14 parts, among them J3 3.5mm_HP_Detect, U4 MAX98357AEWL+T

Commit message: Add kicad/audio_output.kicad_sch
Parts:
- added C35: 22uF/10V X5R, Capacitor_SMD:C_0805_2012Metric, symbol Device:C
- added FB1: 220R@100MHz 500mA, Inductor_SMD:L_0402_1005Metric, symbol Device:Ferrite_Bead
- C22: value 10uF/10V -> 10uF/10V X5R
- C_HP_L, C_HP_R: value 100uF/10V -> 47uF/10V X5R; footprint Capacitor_SMD:CP_Elec_4x5.4 -> Capacitor_SMD:C_0805_2012Metric
- SPK1: value 8Ω/1W/1511 -> 8Ohm/1W/20mm
Other:
- note added: "AUDIO OUTPUT NOTES (v1.1): 1) MAX98357A I2S Class-D: BCLK=IO18, LRCK=IO19, DIN=AMP_I2S_DOUT (separate I2S port from ES7243E) SD_MODE = AMP_SD (IO33): HIGH=left ch play, LOW=shutdown, FLOAT=mono mix Firmware: set LOW when BT connected, HIGH when disconnected 2) PVDD power path: VBAT → FB1(220Ω@100MHz ferrite, 0402) → C35(22uF 0805) → PVDD_FILT → C22(10uF 0805) + C21(100nF 0402) → U4 PVDD [FIXED] F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"
- note removed: "AUDIO OUTPUT DESIGN NOTES: 1) MAX98357A receives I2S from ESP32 (separate I2S port from ES7243E ADC) ESP32 plays decoded/passthrough audio back via I2S DAC port BCLK/LRCK shared with ES7243E but data lines are separate SD_MODE = HIGH → Left channel output only (mono speaker) SD_MODE = LOW → Amplifier shutdown (BT connected = speaker mute) SD_MODE = FLOAT → Left+Right mix to mono (use for mono spe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"
